File: layouts/lightplay2/lightplay2.brd (EAGLE design)
At the start: 81 x 64.8 mm, 51 parts, among them Q0 MOSFET-NCHANNELAO3404A, Q1 MOSFET-NCHANNELAO3404A, Q10 MOSFET-NCHANNELAO3404A, Q11 MOSFET-NCHANNELAO3404A, Q2 MOSFET-NCHANNELAO3404A, Q4 MOSFET-NCHANNELAO3404A, Q5 MOSFET-NCHANNELAO3404A, Q6 MOSFET-NCHANNELAO3404A, Q7 MOSFET-NCHANNELAO3404A, Q8 MOSFET-NCHANNELAO3404A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

Commit message: updated layout files
Parts:
- R16, R17: value 10k -> 1k
- U2: device robbie:SO28W -> robbie:TSSOP28
- moved R16 19.2 mm to (16.5, 15.2)
- moved R17 19.1 mm to (16.5, 10.2)
- moved R18 12.7 mm to (35.6, 17.8)
- moved U2 2.54 mm to (39.4, 29.2), turned to 270 degrees
- moved U1 1.27 mm to (63.5, 30.5)
Connections:
- new net +3V3: ARDUINOLEFT.4, R16.2, R17.2, R18.2, U2.24, U2.28, U2.5
- net +5V: now also LIGHT1.5, LIGHT2.5, LIGHT3.5; no longer R16.2, R17.2, R18.2, U2.28
- net GND: no longer U2.24, U2.5
Routing:
- net LED3: track 99.7 -> 22.6 mm, vias 4 -> 2
- net +3V3: track 0.00 -> 74.9 mm, vias 0 -> 5
- net LED6: track 74.1 -> 18.9 mm, vias 8 -> 0
- net A1: track 128.7 -> 80.8 mm
- net +5V: track 282.5 -> 245.6 mm, vias 1 -> 2
- net D7: track 74.6 -> 38.0 mm, vias 3 -> 0
- net LED2: track 59.2 -> 28.0 mm, vias 6 -> 2
- net SCL: track 84.5 -> 54.9 mm, vias 3 -> 1
- net GND: track 327.7 -> 353.9 mm
- net D2: track 55.5 -> 31.5 mm
- net PWM6: track 67.4 -> 53.7 mm, vias 3 -> 1
- net A0: track 91.3 -> 80.1 mm, vias 2 -> 0
- net LED8: track 8.77 -> 19.6 mm
- net LED9: track 14.9 -> 25.2 mm, vias 0 -> 2
- net LED5: track 29.4 -> 19.8 mm
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