File: layouts/lightplay2/lightplay2.sch (EAGLE design)
At the start: 51 parts, among them Q0 MOSFET-NCHANNELAO3404A, Q1 MOSFET-NCHANNELAO3404A, Q10 MOSFET-NCHANNELAO3404A, Q11 MOSFET-NCHANNELAO3404A, Q2 MOSFET-NCHANNELAO3404A, Q3 MOSFET-NCHANNELAO3404A, Q4 MOSFET-NCHANNELAO3404A, Q5 MOSFET-NCHANNELAO3404A, Q6 MOSFET-NCHANNELAO3404A, Q7 MOSFET-NCHANNELAO3404A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

Commit message: updated layout files
Parts:
- R16, R17: value 10k -> 1k
Connections:
- new net +3V3: ARDUINOLEFT.4, R16.2, R17.2, R18.2, U2.A4, U2.A5, U2.VDD
- net +5V: now also LIGHT1.5, LIGHT2.5, LIGHT3.5; no longer R16.2, R17.2, R18.2, U2.VDD
- net GND: no longer U2.A4, U2.A5
