File: layouts/lightplay2a/lightplay2a.sch (EAGLE design)
At the start: 55 parts, among them Q0 MOSFET-NCHANNELAO3404A, Q1 MOSFET-NCHANNELAO3404A, Q10 MOSFET-NCHANNELAO3404A, Q11 MOSFET-NCHANNELAO3404A, Q2 MOSFET-NCHANNELAO3404A, Q3 MOSFET-NCHANNELAO3404A, Q4 MOSFET-NCHANNELAO3404A, Q5 MOSFET-NCHANNELAO3404A, Q6 MOSFET-NCHANNELAO3404A, Q7 MOSFET-NCHANNELAO3404A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

Commit message: working on Arduino code for LightPlay2a
Parts:
- U3: value STM3.3VREG -> 3.3VREG
- renumbered U$1 to U3
Changed lines of the file:
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@@
 <part name="+3V5" library="supply1" deviceset="+3V3" device=""/>
 <part name="C6" library="resistor" deviceset="C-US" device="C0805" value="0.1uF"/>
-<part name="U$1" library="robbie" deviceset="STM3.3VREG" device=""/>
+<part name="U3" library="robbie" deviceset="STM3.3VREG" device="" value="3.3VREG"/>
 <part name="P+5" library="supply1" deviceset="+5V" device=""/>
 <part name="+3V6" library="supply1" deviceset="+3V3" device=""/>
@@
 <instance part="+3V5" gate="G$1" x="-76.2" y="20.32"/>
 <instance part="C6" gate="G$1" x="-60.96" y="12.7"/>
-<instance part="U$1" gate="G$1" x="-58.42" y="-88.9"/>
+<instance part="U3" gate="G$1" x="-58.42" y="-88.9"/>
 <instance part="P+5" gate="1" x="-66.04" y="-73.66"/>
 <instance part="+3V6" gate="G$1" x="-81.28" y="-73.66"/>
@@
 </segment>
 <segment>
-<pinref part="U$1" gate="G$1" pin="GND"/>
+<pinref part="U3" gate="G$1" pin="GND"/>
 <wire x1="-63.5" y1="-88.9" x2="-66.04" y2="-88.9" width="0.1524" layer="91"/>
 <pinref part="GND31" gate="1" pin="GND"/>
@@
 </segment>
 <segment>
-<pinref part="U$1" gate="G$1" pin="VIN"/>
+<pinref part="U3" gate="G$1" pin="VIN"/>
 <wire x1="-63.5" y1="-83.82" x2="-66.04" y2="-83.82" width="0.1524" layer="91"/>
 <pinref part="P+5" gate="1" pin="+5V"/>
@@
 </segment>
 <segment>
-<pinref part="U$1" gate="G$1" pin="VOUT"/>
+<pinref part="U3" gate="G$1" pin="VOUT"/>
 <wire x1="-63.5" y1="-93.98" x2="-81.28" y2="-93.98" width="0.1524" layer="91"/>
 <pinref part="+3V6" gate="G$1" pin="+3V3"/>

Commit message: updated Blocks documentation to include new command numbers to avoid sending '+' character to Bluetooth UART
Parts:
- C8: value 0.1uF -> TDB
Changed lines of the file:
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@@
 <part name="GND31" library="supply1" deviceset="GND" device=""/>
 <part name="C7" library="resistor" deviceset="C-US" device="C1206" value="0.33 uF"/>
-<part name="C8" library="resistor" deviceset="C-US" device="C0805" value="0.1uF"/>
+<part name="C8" library="resistor" deviceset="C-US" device="C0805" value="TDB"/>
 <part name="GND32" library="supply1" deviceset="GND" device=""/>
 <part name="C2" library="resistor" deviceset="C-US" device="C0805" value="0.1uF"/>
